Commit message: I broke something

File: body.urdf (robot description, URDF)
Before this commit: robot robot, 7 links, 6 joints
Links:
- removed link Link0
- removed link Link1
- removed link Link2
- removed link Link3
- removed link Link4
- removed link Link5
- removed link Link6
- added link BackLeg, mass 1; collision box size=0.2 1 0.2; visual box size=0.2 1 0.2
- added link FrontLeg, mass 1; collision box size=0.2 1 0.2; visual box size=0.2 1 0.2
- added link LeftLeg, mass 1; collision box size=1 0.2 0.2; visual box size=1 0.2 0.2
- added link LowerBackLeg, mass 1; collision box size=0.2 0.2 1; visual box size=0.2 0.2 1
- added link LowerFrontLeg, mass 1; collision box size=0.2 0.2 1; visual box size=0.2 0.2 1
- added link LowerLeftLeg, mass 1; collision box size=0.2 0.2 1; visual box size=0.2 0.2 1
- added link LowerRightLeg, mass 1; collision box size=0.2 0.2 1; visual box size=0.2 0.2 1
- added link RightLeg, mass 1; collision box size=1 0.2 0.2; visual box size=1 0.2 0.2
- added link Torso, mass 1; collision box size=1 1 1; visual box size=1 1 1
Joints:
- removed joint Link0_Link1
- removed joint Link1_Link2
- removed joint Link2_Link3
- removed joint Link3_Link4
- removed joint Link4_Link5
- removed joint Link5_Link6
- added joint BackLeg_LowerBackLeg: type revolute, parent BackLeg, child LowerBackLeg, origin xyz=0 -1 0 rpy=0 0 0, axis 1 0 0, limit lower=-3.14159 upper=3.14159 effort=0.0 velocity=0.0
- added joint FrontLeg_LowerFrontLeg: type revolute, parent FrontLeg, child LowerFrontLeg, origin xyz=0 1 0 rpy=0 0 0, axis 1 0 0, limit lower=-3.14159 upper=3.14159 effort=0.0 velocity=0.0
- added joint LeftLeg_LowerLeftLeg: type revolute, parent LeftLeg, child LowerLeftLeg, origin xyz=-1 0 0 rpy=0 0 0, axis 0 1 0, limit lower=-3.14159 upper=3.14159 effort=0.0 velocity=0.0
- added joint RightLeg_LowerRightLeg: type revolute, parent RightLeg, child LowerRightLeg, origin xyz=1 0 0 rpy=0 0 0, axis 0 1 0, limit lower=-3.14159 upper=3.14159 effort=0.0 velocity=0.0
- added joint Torso_BackLeg: type revolute, parent Torso, child BackLeg, origin xyz=0 -0.5 1 rpy=0 0 0, axis 1 0 0, limit lower=-3.14159 upper=3.14159 effort=0.0 velocity=0.0
- added joint Torso_FrontLeg: type revolute, parent Torso, child FrontLeg, origin xyz=0 0.5 1 rpy=0 0 0, axis 1 0 0, limit lower=-3.14159 upper=3.14159 effort=0.0 velocity=0.0
- added joint Torso_LeftLeg: type revolute, parent Torso, child LeftLeg, origin xyz=-0.5 0 1 rpy=0 0 0, axis 0 1 0, limit lower=-3.14159 upper=3.14159 effort=0.0 velocity=0.0
- added joint Torso_RightLeg: type revolute, parent Torso, child RightLeg, origin xyz=0.5 0 1 rpy=0 0 0, axis 0 1 0, limit lower=-3.14159 upper=3.14159 effort=0.0 velocity=0.0

Commit message: Working on dog body

File: body.urdf (robot description, URDF)
Before this commit: robot robot, 9 links, 8 joints
Links:
- removed link BackLeg
- removed link FrontLeg
- removed link LeftLeg
- removed link LowerBackLeg
- removed link LowerLeftLeg
- removed link LowerRightLeg
- removed link RightLeg
- added link BackLeftLeg, mass 1; collision box size=0.2 1 0.2; visual box size=0.2 1 0.2
- added link BackRightLeg, mass 1; collision box size=1 0.2 0.2; visual box size=1 0.2 0.2
- added link FrontLeftLeg, mass 1; collision box size=0.2 1 0.2; visual box size=0.2 1 0.2
- added link FrontRightLeg, mass 1; collision box size=1 0.2 0.2; visual box size=1 0.2 0.2
- added link LowerBackLeftLeg, mass 1; collision box size=0.2 0.2 1; visual box size=0.2 0.2 1
- added link LowerBackRightLeg, mass 1; collision box size=0.2 0.2 1; visual box size=0.2 0.2 1
- added link LowerFrontRightLeg, mass 1; collision box size=0.2 0.2 1; visual box size=0.2 0.2 1
- link Torso: geometry collision box size=2 0.8 1; visual box size=2 0.8 1
Joints:
- removed joint BackLeg_LowerBackLeg
- removed joint FrontLeg_LowerFrontLeg
- removed joint LeftLeg_LowerLeftLeg
- removed joint RightLeg_LowerRightLeg
- removed joint Torso_BackLeg
- removed joint Torso_FrontLeg
- removed joint Torso_LeftLeg
- removed joint Torso_RightLeg
- added joint BackLeftLeg_LowerBackLeftLeg: type revolute, parent BackLeftLeg, child LowerBackLeftLeg, origin xyz=-0.5 0 -1 rpy=0 0 0, axis 1 0 0, limit lower=-3.14159 upper=3.14159 effort=0.0 velocity=0.0
- added joint BackRightLeg_LowerBackRightLeg: type revolute, parent BackRightLeg, child LowerBackRightLeg, origin xyz=0.5 0 -1 rpy=0 0 0, axis 0 1 0, limit lower=-3.14159 upper=3.14159 effort=0.0 velocity=0.0
- added joint FrontLeftLeg_LowerFrontLeftLeg: type revolute, parent FrontLeftLeg, child LowerFrontLeftLeg, origin xyz=-0.5 0 -1 rpy=0 0 0, axis 1 0 0, limit lower=-3.14159 upper=3.14159 effort=0.0 velocity=0.0
- added joint FrontRightLeg_LowerFrontRightLeg: type revolute, parent FrontRightLeg, child LowerFrontRightLeg, origin xyz=0.5 0 -1 rpy=0 0 0, axis 0 1 0, limit lower=-3.14159 upper=3.14159 effort=0.0 velocity=0.0
- added joint Torso_BackLeftLeg: type revolute, parent Torso, child BackLeftLeg, origin xyz=-0.5 -0.5 1.5 rpy=0 0 0, axis 1 0 0, limit lower=-3.14159 upper=3.14159 effort=0.0 velocity=0.0
- added joint Torso_BackRightLeg: type revolute, parent Torso, child BackRightLeg, origin xyz=0.5 -0.5 1.5 rpy=0 0 0, axis 0 1 0, limit lower=-3.14159 upper=3.14159 effort=0.0 velocity=0.0
- added joint Torso_FrontLeftLeg: type revolute, parent Torso, child FrontLeftLeg, origin xyz=-0.5 0.5 1.5 rpy=0 0 0, axis 1 0 0, limit lower=-3.14159 upper=3.14159 effort=0.0 velocity=0.0
- added joint Torso_FrontRightLeg: type revolute, parent Torso, child FrontRightLeg, origin xyz=0.5 0.5 1.5 rpy=0 0 0, axis 0 1 0, limit lower=-3.14159 upper=3.14159 effort=0.0 velocity=0.0

Commit message: Fixed it, if it breaks again, make sure self.robotId isn't self.robot in robot.py on line 34

File: body.urdf (robot description, URDF)
Before this commit: robot robot, 9 links, 8 joints
Links:
- removed link BackLeftLeg
- removed link BackRightLeg
- removed link FrontLeftLeg
- removed link FrontRightLeg
- removed link LowerBackLeftLeg
- removed link LowerBackRightLeg
- removed link LowerFrontRightLeg
- added link BackLeg, mass 1; collision box size=0.2 1 0.2; visual box size=0.2 1 0.2
- added link FrontLeg, mass 1; collision box size=0.2 1 0.2; visual box size=0.2 1 0.2
- added link LeftLeg, mass 1; collision box size=1 0.2 0.2; visual box size=1 0.2 0.2
- added link LowerBackLeg, mass 1; collision box size=0.2 0.2 1; visual box size=0.2 0.2 1
- added link LowerLeftLeg, mass 1; collision box size=0.2 0.2 1; visual box size=0.2 0.2 1
- added link LowerRightLeg, mass 1; collision box size=0.2 0.2 1; visual box size=0.2 0.2 1
- added link RightLeg, mass 1; collision box size=1 0.2 0.2; visual box size=1 0.2 0.2
- link Torso: geometry collision box size=1 1 1; visual box size=1 1 1
Joints:
- removed joint BackLeftLeg_LowerBackLeftLeg
- removed joint BackRightLeg_LowerBackRightLeg
- removed joint FrontLeftLeg_LowerFrontLeftLeg
- removed joint FrontRightLeg_LowerFrontRightLeg
- removed joint Torso_BackLeftLeg
- removed joint Torso_BackRightLeg
- removed joint Torso_FrontLeftLeg
- removed joint Torso_FrontRightLeg
- added joint BackLeg_LowerBackLeg: type revolute, parent BackLeg, child LowerBackLeg, origin xyz=0 -1 0 rpy=0 0 0, axis 1 0 0, limit lower=-3.14159 upper=3.14159 effort=0.0 velocity=0.0
- added joint FrontLeg_LowerFrontLeg: type revolute, parent FrontLeg, child LowerFrontLeg, origin xyz=0 1 0 rpy=0 0 0, axis 1 0 0, limit lower=-3.14159 upper=3.14159 effort=0.0 velocity=0.0
- added joint LeftLeg_LowerLeftLeg: type revolute, parent LeftLeg, child LowerLeftLeg, origin xyz=-1 0 0 rpy=0 0 0, axis 0 1 0, limit lower=-3.14159 upper=3.14159 effort=0.0 velocity=0.0
- added joint RightLeg_LowerRightLeg: type revolute, parent RightLeg, child LowerRightLeg, origin xyz=1 0 0 rpy=0 0 0, axis 0 1 0, limit lower=-3.14159 upper=3.14159 effort=0.0 velocity=0.0
- added joint Torso_BackLeg: type revolute, parent Torso, child BackLeg, origin xyz=0 -0.5 1 rpy=0 0 0, axis 1 0 0, limit lower=-3.14159 upper=3.14159 effort=0.0 velocity=0.0
- added joint Torso_FrontLeg: type revolute, parent Torso, child FrontLeg, origin xyz=0 0.5 1 rpy=0 0 0, axis 1 0 0, limit lower=-3.14159 upper=3.14159 effort=0.0 velocity=0.0
- added joint Torso_LeftLeg: type revolute, parent Torso, child LeftLeg, origin xyz=-0.5 0 1 rpy=0 0 0, axis 0 1 0, limit lower=-3.14159 upper=3.14159 effort=0.0 velocity=0.0
- added joint Torso_RightLeg: type revolute, parent Torso, child RightLeg, origin xyz=0.5 0 1 rpy=0 0 0, axis 0 1 0, limit lower=-3.14159 upper=3.14159 effort=0.0 velocity=0.0

Commit message: Spot robot

File: body.urdf (robot description, URDF)
Before this commit: robot robot, 9 links, 8 joints
Links:
- link BackLeg: geometry collision box size=0.2 0.2 0.5; visual box size=0.2 0.2 0.5
- link FrontLeg: geometry collision box size=0.2 0.2 0.5; visual box size=0.2 0.2 0.5
- link LeftLeg: geometry collision box size=0.2 0.2 0.5; visual box size=0.2 0.2 0.5
- link LowerBackLeg: geometry collision box size=0.2 0.2 0.5; visual box size=0.2 0.2 0.5
- link LowerFrontLeg: geometry collision box size=0.2 0.2 0.5; visual box size=0.2 0.2 0.5
- link LowerLeftLeg: geometry collision box size=0.2 0.2 0.5; visual box size=0.2 0.2 0.5
- link LowerRightLeg: geometry collision box size=0.2 0.2 0.5; visual box size=0.2 0.2 0.5
- link RightLeg: geometry collision box size=0.2 0.2 0.5; visual box size=0.2 0.2 0.5
- link Torso: geometry collision box size=1.8 0.8 0.4; visual box size=1.8 0.8 0.4
Joints:
- joint BackLeg_LowerBackLeg: axis 1 0 0 -> 0 1 0; origin xyz=0 -1 0 rpy=0 0 0 -> xyz=0 -0.5 -0.2 rpy=0 0 0
- joint FrontLeg_LowerFrontLeg: axis 1 0 0 -> 0 1 0; origin xyz=0 1 0 rpy=0 0 0 -> xyz=0 -0.5 -0.25 rpy=0 0 0
- joint LeftLeg_LowerLeftLeg: origin xyz=-1 0 0 rpy=0 0 0 -> xyz=0 0.5 -0.2 rpy=0 0 0
- joint RightLeg_LowerRightLeg: origin xyz=1 0 0 rpy=0 0 0 -> xyz=0 0.5 -0.2 rpy=0 0 0
- joint Torso_BackLeg: axis 1 0 0 -> 0 1 0; origin xyz=0 -0.5 1 rpy=0 0 0 -> xyz=0.5 0 2 rpy=0 0 0
- joint Torso_FrontLeg: axis 1 0 0 -> 0 1 0; origin xyz=0 0.5 1 rpy=0 0 0 -> xyz=-0.5 0 2 rpy=0 0 0
- joint Torso_LeftLeg: origin xyz=-0.5 0 1 rpy=0 0 0 -> xyz=-0.5 0 2 rpy=0 0 0
- joint Torso_RightLeg: origin xyz=0.5 0 1 rpy=0 0 0 -> xyz=0.5 0 2 rpy=0 0 0

Commit message: Basic arm prototype

File: body.urdf (robot description, URDF)
Before this commit: robot robot, 9 links, 8 joints
Links:
- added link LowerArm, mass 1; collision box size=0.2 0.2 0.8; visual box size=0.2 0.2 0.8
- added link UpperArm, mass 1; collision box size=0.8 0.2 0.2; visual box size=0.8 0.2 0.2
Joints:
- added joint LowerArm_UpperArm: type revolute, parent LowerArm, child UpperArm, origin xyz=0 0 0.8 rpy=0 0 0, axis 0 1 0, limit lower=-3.14159 upper=3.14159 effort=0.0 velocity=0.0
- added joint Torso_LowerArm: type revolute, parent Torso, child LowerArm, origin xyz=-0.5 0 2.1 rpy=0 0 0, axis 0 1 0, limit lower=-3.14159 upper=3.14159 effort=0.0 velocity=0.0

Commit message: Finger prototype

File: body.urdf (robot description, URDF)
Before this commit: robot robot, 11 links, 10 joints
Links:
- added link BottomFinger, mass 1; collision box size=0.4 0.2 0.1; visual box size=0.4 0.2 0.1
- added link TopFinger, mass 1; collision box size=0.4 0.2 0.1; visual box size=0.4 0.2 0.1
Joints:
- added joint UpperArm_BottomFinger: type revolute, parent UpperArm, child BottomFinger, origin xyz=-0.8 0 -0.1 rpy=0 0 0, axis 0 1 0, limit lower=-3.14159 upper=3.14159 effort=0.0 velocity=0.0
- added joint UpperArm_TopFinger: type revolute, parent UpperArm, child TopFinger, origin xyz=-0.8 0 0.1 rpy=0 0 0, axis 0 1 0, limit lower=-3.14159 upper=3.14159 effort=0.0 velocity=0.0

Commit message: Updated brain, need to ask for advice on making bot move more than it currently is

File: body.urdf (robot description, URDF)
Before this commit: robot robot, 13 links, 12 joints
Joints:
- joint BackLeg_LowerBackLeg: origin xyz=0 -0.5 -0.2 rpy=0 0 0 -> xyz=0.1 -0.5 -0.2 rpy=0 0 0
- joint FrontLeg_LowerFrontLeg: origin xyz=0 -0.5 -0.25 rpy=0 0 0 -> xyz=-0.1 -0.5 -0.25 rpy=0 0 0
- joint LeftLeg_LowerLeftLeg: origin xyz=0 0.5 -0.2 rpy=0 0 0 -> xyz=-0.1 0.5 -0.2 rpy=0 0 0
- joint RightLeg_LowerRightLeg: origin xyz=0 0.5 -0.2 rpy=0 0 0 -> xyz=0.1 0.5 -0.2 rpy=0 0 0

Commit message: Baseline: has file output for each generation's best fitness working, testing runs both cases sequentially

File: body.urdf (robot description, URDF)
Before this commit: robot robot, 13 links, 12 joints
Links:
- removed link BottomFinger
- removed link LowerArm
- removed link TopFinger
- removed link UpperArm
- link BackLeg: geometry collision box size=0.2 1 0.2; visual box size=0.2 1 0.2
- link FrontLeg: geometry collision box size=0.2 1 0.2; visual box size=0.2 1 0.2
- link LeftLeg: geometry collision box size=1 0.2 0.2; visual box size=1 0.2 0.2
- link LowerBackLeg: geometry collision box size=0.2 0.2 1; visual box size=0.2 0.2 1
- link LowerFrontLeg: geometry collision box size=0.2 0.2 1; visual box size=0.2 0.2 1
- link LowerLeftLeg: geometry collision box size=0.2 0.2 1; visual box size=0.2 0.2 1
- link LowerRightLeg: geometry collision box size=0.2 0.2 1; visual box size=0.2 0.2 1
- link RightLeg: geometry collision box size=1 0.2 0.2; visual box size=1 0.2 0.2
- link Torso: geometry collision box size=1 1 1; visual box size=1 1 1
Joints:
- removed joint LowerArm_UpperArm
- removed joint Torso_LowerArm
- removed joint UpperArm_BottomFinger
- removed joint UpperArm_TopFinger
- joint BackLeg_LowerBackLeg: axis 0 1 0 -> 1 0 0; origin xyz=0.1 -0.5 -0.2 rpy=0 0 0 -> xyz=0 -1 0 rpy=0 0 0
- joint FrontLeg_LowerFrontLeg: axis 0 1 0 -> 1 0 0; origin xyz=-0.1 -0.5 -0.25 rpy=0 0 0 -> xyz=0 1 0 rpy=0 0 0
- joint LeftLeg_LowerLeftLeg: origin xyz=-0.1 0.5 -0.2 rpy=0 0 0 -> xyz=-1 0 0 rpy=0 0 0
- joint RightLeg_LowerRightLeg: origin xyz=0.1 0.5 -0.2 rpy=0 0 0 -> xyz=1 0 0 rpy=0 0 0
- joint Torso_BackLeg: axis 0 1 0 -> 1 0 0; origin xyz=0.5 0 2 rpy=0 0 0 -> xyz=0 -0.5 1 rpy=0 0 0
- joint Torso_FrontLeg: axis 0 1 0 -> 1 0 0; origin xyz=-0.5 0 2 rpy=0 0 0 -> xyz=0 0.5 1 rpy=0 0 0
- joint Torso_LeftLeg: origin xyz=-0.5 0 2 rpy=0 0 0 -> xyz=-0.5 0 1 rpy=0 0 0
- joint Torso_RightLeg: origin xyz=0.5 0 2 rpy=0 0 0 -> xyz=0.5 0 1 rpy=0 0 0

Commit message: Changed b version to be same body but without recurrent synaptic connections

File: body.urdf (robot description, URDF)
Before this commit: robot robot, 9 links, 8 joints
Links:
- added link BottomFinger, mass 1; collision box size=0.4 0.2 0.1; visual box size=0.4 0.2 0.1
- added link LowerArm, mass 1; collision box size=0.2 0.2 0.8; visual box size=0.2 0.2 0.8
- added link TopFinger, mass 1; collision box size=0.4 0.2 0.1; visual box size=0.4 0.2 0.1
- added link UpperArm, mass 1; collision box size=0.8 0.2 0.2; visual box size=0.8 0.2 0.2
- link BackLeg: geometry collision box size=0.2 0.2 0.5; visual box size=0.2 0.2 0.5
- link FrontLeg: geometry collision box size=0.2 0.2 0.5; visual box size=0.2 0.2 0.5
- link LeftLeg: geometry collision box size=0.2 0.2 0.5; visual box size=0.2 0.2 0.5
- link LowerBackLeg: geometry collision box size=0.2 0.2 0.5; visual box size=0.2 0.2 0.5
- link LowerFrontLeg: geometry collision box size=0.2 0.2 0.5; visual box size=0.2 0.2 0.5
- link LowerLeftLeg: geometry collision box size=0.2 0.2 0.5; visual box size=0.2 0.2 0.5
- link LowerRightLeg: geometry collision box size=0.2 0.2 0.5; visual box size=0.2 0.2 0.5
- link RightLeg: geometry collision box size=0.2 0.2 0.5; visual box size=0.2 0.2 0.5
- link Torso: geometry collision box size=1.8 0.8 0.4; visual box size=1.8 0.8 0.4
Joints:
- added joint LowerArm_UpperArm: type revolute, parent LowerArm, child UpperArm, origin xyz=0 0 0.8 rpy=0 0 0, axis 0 1 0, limit lower=-3.14159 upper=3.14159 effort=0.0 velocity=0.0
- added joint Torso_LowerArm: type revolute, parent Torso, child LowerArm, origin xyz=-0.5 0 2.1 rpy=0 0 0, axis 0 1 0, limit lower=-3.14159 upper=3.14159 effort=0.0 velocity=0.0
- added joint UpperArm_BottomFinger: type revolute, parent UpperArm, child BottomFinger, origin xyz=-0.8 0 -0.1 rpy=0 0 0, axis 0 1 0, limit lower=-3.14159 upper=3.14159 effort=0.0 velocity=0.0
- added joint UpperArm_TopFinger: type revolute, parent UpperArm, child TopFinger, origin xyz=-0.8 0 0.1 rpy=0 0 0, axis 0 1 0, limit lower=-3.14159 upper=3.14159 effort=0.0 velocity=0.0
- joint BackLeg_LowerBackLeg: axis 1 0 0 -> 0 1 0; origin xyz=0 -1 0 rpy=0 0 0 -> xyz=0.1 -0.5 -0.2 rpy=0 0 0
- joint FrontLeg_LowerFrontLeg: axis 1 0 0 -> 0 1 0; origin xyz=0 1 0 rpy=0 0 0 -> xyz=-0.1 -0.5 -0.25 rpy=0 0 0
- joint LeftLeg_LowerLeftLeg: origin xyz=-1 0 0 rpy=0 0 0 -> xyz=-0.1 0.5 -0.2 rpy=0 0 0
- joint RightLeg_LowerRightLeg: origin xyz=1 0 0 rpy=0 0 0 -> xyz=0.1 0.5 -0.2 rpy=0 0 0
- joint Torso_BackLeg: axis 1 0 0 -> 0 1 0; origin xyz=0 -0.5 1 rpy=0 0 0 -> xyz=0.5 0 2 rpy=0 0 0
- joint Torso_FrontLeg: axis 1 0 0 -> 0 1 0; origin xyz=0 0.5 1 rpy=0 0 0 -> xyz=-0.5 0 2 rpy=0 0 0
- joint Torso_LeftLeg: origin xyz=-0.5 0 1 rpy=0 0 0 -> xyz=-0.5 0 2 rpy=0 0 0
- joint Torso_RightLeg: origin xyz=0.5 0 1 rpy=0 0 0 -> xyz=0.5 0 2 rpy=0 0 0
